File: PWM_.sch (EAGLE design)
At the start: 9 parts, among them IC1 LM555D

Commit message: updated to match all the pinouts
left, right, front, back, connections consistent PWM added to the light boards
Changed lines of the file:
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@@
 <segment>
 <pinref part="IC1" gate="A" pin="TR"/>
-<wire x1="-10.16" y1="7.62" x2="-12.7" y2="7.62" width="0.1524" layer="91"/>
 <pinref part="GND4" gate="1" pin="GND"/>
-<wire x1="-12.7" y1="7.62" x2="-12.7" y2="12.7" width="0.1524" layer="91"/>
+<wire x1="-10.16" y1="7.62" x2="-12.7" y2="12.7" width="0.1524" layer="91"/>
 </segment>
 <segment>
