File: Font _light_connect.brd (EAGLE design)
At the start: 59.8 x 72.7 mm, 5 parts

Commit message: all gerbers generated
Parts:
- added H1, H2, H3, H4: STAND-OFF, SparkFun-Electromechanical:STAND-OFF
Changed lines of the file:
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@@
 <element name="R_SIG" library="TE 2-pin connector" package="2_PIN_CONNECT" value="2_PIN_TECONNECTOR" x="90.17" y="48.26" rot="R90"/>
 <element name="T_DRIVE" library="TE 2-pin connector" package="2_PIN_CONNECT" value="2_PIN_TECONNECTOR" x="90.17" y="13.97" rot="R90"/>
+<element name="H1" library="SparkFun-Electromechanical" package="STAND-OFF" value="STAND-OFF" x="44.1" y="5.775"/>
+<element name="H2" library="SparkFun-Electromechanical" package="STAND-OFF" value="STAND-OFF" x="96.25" y="5.775"/>
+<element name="H3" library="SparkFun-Electromechanical" package="STAND-OFF" value="STAND-OFF" x="44.1" y="70.7"/>
+<element name="H4" library="SparkFun-Electromechanical" package="STAND-OFF" value="STAND-OFF" x="96.425" y="70.7"/>
 </elements>
 <signals>
