File: Font _light_connect.sch (EAGLE design)
At the start: 5 parts

Commit message: updated to match all the pinouts
left, right, front, back, connections consistent PWM added to the light boards
Parts:
- removed U$1, U$2, U$3, U$4: 43650-0200, Shell2013:43650-0200
- added L_DRIVE, L_SIG, R_SIG, T_DRIVE: 2_PIN_TECONNECTOR, TE 2-pin connector:2_PIN_TECONNECTOR
- renumbered ETH1 to REAR
Connections:
- net N$1: now also L_DRIVE.V/SIG; no longer U$4.P$2
- net N$2: now also L_SIG.V/SIG; no longer U$4.P$1
- net N$3: now also REAR.5, R_SIG.V/SIG; no longer REAR.3, U$3.P$2
- net N$4: now also L_SIG.G/LOW; no longer U$3.P$1
- net N$5: now also L_DRIVE.G/LOW, REAR.7; no longer REAR.5, U$2.P$2
- net N$6: now also R_SIG.G/LOW; no longer U$2.P$1
- net N$7: now also REAR.3, T_DRIVE.V/SIG; no longer REAR.7, U$1.P$2
- net N$8: now also T_DRIVE.G/LOW; no longer U$1.P$1
Changed lines of the file:
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@@
 <?xml version="1.0" encoding="utf-8"?>
 <!DOCTYPE eagle SYSTEM "eagle.dtd">
-<eagle version="8.4.2">
+<eagle version="8.3.1">
 <drawing>
 <settings>
@@
 </classes>
 <parts>
-<part name="U$1" library="Shell2013" deviceset="43650-0200" device=""/>
-<part name="U$2" library="Shell2013" deviceset="43650-0200" device=""/>
-<part name="U$3" library="Shell2013" deviceset="43650-0200" device=""/>
-<part name="U$4" library="Shell2013" deviceset="43650-0200" device=""/>
-<part name="ETH1" library="ETHERNET" deviceset="ETHERNET" device=""/>
+<part name="REAR" library="ETHERNET" deviceset="ETHERNET" device=""/>
+<part name="T_DRIVE" library="TE 2-pin connector" deviceset="2_PIN_TECONNECTOR" device=""/>
+<part name="R_SIG" library="TE 2-pin connector" deviceset="2_PIN_TECONNECTOR" device=""/>
+<part name="L_SIG" library="TE 2-pin connector" deviceset="2_PIN_TECONNECTOR" device=""/>
+<part name="L_DRIVE" library="TE 2-pin connector" deviceset="2_PIN_TECONNECTOR" device=""/>
 </parts>
 <sheets>
@@
 </plain>
 <instances>
-<instance part="U$1" gate="G$1" x="107.95" y="87.63"/>
-<instance part="U$2" gate="G$1" x="107.95" y="69.85"/>
-<instance part="U$3" gate="G$1" x="107.95" y="50.8"/>
-<instance part="U$4" gate="G$1" x="107.95" y="30.48"/>
-<instance part="ETH1" gate="G$1" x="48.26" y="68.58" rot="R180"/>
+<instance part="REAR" gate="G$1" x="48.26" y="68.58" rot="R180"/>
+<instance part="T_DRIVE" gate="G$1" x="116.84" y="88.9"/>
+<instance part="R_SIG" gate="G$1" x="119.38" y="68.58"/>
+<instance part="L_SIG" gate="G$1" x="119.38" y="50.8"/>
+<instance part="L_DRIVE" gate="G$1" x="119.38" y="30.48"/>
 </instances>
 <busses>
@@
 <net name="N$1" class="0">
 <segment>
-<pinref part="ETH1" gate="G$1" pin="1"/>
+<pinref part="REAR" gate="G$1" pin="1"/>
 <wire x1="53.34" y1="53.34" x2="63.5" y2="53.34" width="0.1524" layer="91"/>
 <wire x1="63.5" y1="53.34" x2="63.5" y2="27.94" width="0.1524" layer="91"/>
-<pinref part="U$4" gate="G$1" pin="P$2"/>
-<wire x1="63.5" y1="27.94" x2="102.87" y2="27.94" width="0.1524" layer="91"/>
-</segment>
-</net>
-<net name="N$2" class="0">
-<segment>
-<pinref part="ETH1" gate="G$1" pin="2"/>
-<wire x1="53.34" y1="55.88" x2="66.04" y2="55.88" width="0.1524" layer="91"/>
-<pinref part="U$4" gate="G$1" pin="P$1"/>
-<wire x1="66.04" y1="55.88" x2="66.04" y2="33.02" width="0.1524" layer="91"/>
-<wire x1="66.04" y1="33.02" x2="102.87" y2="33.02" width="0.1524" layer="91"/>
-</segment>
-</net>
-<net name="N$3" class="0">
-<segment>
-<pinref part="ETH1" gate="G$1" pin="3"/>
-<wire x1="53.34" y1="58.42" x2="71.12" y2="58.42" width="0.1524" layer="91"/>
-<pinref part="U$3" gate="G$1" pin="P$2"/>
-<wire x1="71.12" y1="58.42" x2="71.12" y2="48.26" width="0.1524" layer="91"/>
-<wire x1="71.12" y1="48.26" x2="102.87" y2="48.26" width="0.1524" layer="91"/>
+<wire x1="63.5" y1="27.94" x2="114.3" y2="27.94" width="0.1524" layer="91"/>
+<pinref part="L_DRIVE" gate="G$1" pin="V/SIG"/>
 </segment>
 </net>
 <net name="N$4" class="0">
 <segment>
-<pinref part="ETH1" gate="G$1" pin="4"/>
+<pinref part="REAR" gate="G$1" pin="4"/>
 <wire x1="53.34" y1="60.96" x2="73.66" y2="60.96" width="0.1524" layer="91"/>
-<pinref part="U$3" gate="G$1" pin="P$1"/>
 <wire x1="73.66" y1="60.96" x2="73.66" y2="53.34" width="0.1524" layer="91"/>
-<wire x1="73.66" y1="53.34" x2="102.87" y2="53.34" width="0.1524" layer="91"/>
-</segment>
-</net>
-<net name="N$5" class="0">
-<segment>
-<pinref part="ETH1" gate="G$1" pin="5"/>
-<pinref part="U$2" gate="G$1" pin="P$2"/>
-<wire x1="53.34" y1="63.5" x2="102.87" y2="63.5" width="0.1524" layer="91"/>
-<wire x1="102.87" y1="63.5" x2="102.87" y2="67.31" width="0.1524" layer="91"/>
+<wire x1="73.66" y1="53.34" x2="101.6" y2="53.34" width="0.1524" layer="91"/>
+<pinref part="L_SIG" gate="G$1" pin="G/LOW"/>
+<wire x1="101.6" y1="53.34" x2="102.87" y2="53.34" width="0.1524" layer="91"/>
+<wire x1="102.87" y1="53.34" x2="114.3" y2="53.34" width="0.1524" layer="91"/>
 </segment>
 </net>
 <net name="N$6" class="0">
 <segment>
-<pinref part="ETH1" gate="G$1" pin="6"/>
+<pinref part="REAR" gate="G$1" pin="6"/>
 <wire x1="53.34" y1="66.04" x2="96.52" y2="66.04" width="0.1524" layer="91"/>
 <wire x1="96.52" y1="66.04" x2="96.52" y2="71.12" width="0.1524" layer="91"/>
-<pinref part="U$2" gate="G$1" pin="P$1"/>
-<wire x1="96.52" y1="71.12" x2="102.87" y2="71.12" width="0.1524" layer="91"/>
-<wire x1="102.87" y1="71.12" x2="102.87" y2="72.39" width="0.1524" layer="91"/>
+<wire x1="96.52" y1="71.12" x2="101.6" y2="71.12" width="0.1524" layer="91"/>
+<pinref part="R_SIG" gate="G$1" pin="G/LOW"/>
+<wire x1="101.6" y1="71.12" x2="102.87" y2="71.12" width="0.1524" layer="91"/>
+<wire x1="102.87" y1="71.12" x2="114.3" y2="71.12" width="0.1524" layer="91"/>
+</segment>
+</net>
+<net name="N$8" class="0">
+<segment>
+<pinref part="REAR" gate="G$1" pin="8"/>
+<wire x1="53.34" y1="71.12" x2="86.36" y2="71.12" width="0.1524" layer="91"/>
+<pinref part="T_DRIVE" gate="G$1" pin="G/LOW"/>
+<wire x1="86.36" y1="71.12" x2="86.36" y2="91.44" width="0.1524" layer="91"/>
+<wire x1="86.36" y1="91.44" x2="111.76" y2="91.44" width="0.1524" layer="91"/>
+</segment>
+</net>
+<net name="N$2" class="0">
+<segment>
+<pinref part="REAR" gate="G$1" pin="2"/>
+<wire x1="53.34" y1="55.88" x2="71.12" y2="55.88" width="0.1524" layer="91"/>
+<wire x1="71.12" y1="55.88" x2="71.12" y2="48.26" width="0.1524" layer="91"/>
+<pinref part="L_SIG" gate="G$1" pin="V/SIG"/>
+<wire x1="71.12" y1="48.26" x2="114.3" y2="48.26" width="0.1524" layer="91"/>
+</segment>
+</net>
+<net name="N$3" class="0">
+<segment>
+<pinref part="REAR" gate="G$1" pin="5"/>
+<wire x1="53.34" y1="63.5" x2="106.68" y2="63.5" width="0.1524" layer="91"/>
+<wire x1="106.68" y1="63.5" x2="106.68" y2="66.04" width="0.1524" layer="91"/>
+<pinref part="R_SIG" gate="G$1" pin="V/SIG"/>
+<wire x1="106.68" y1="66.04" x2="114.3" y2="66.04" width="0.1524" layer="91"/>
+</segment>
+</net>
+<net name="N$5" class="0">
+<segment>
+<pinref part="REAR" gate="G$1" pin="7"/>
+<wire x1="53.34" y1="68.58" x2="58.42" y2="68.58" width="0.1524" layer="91"/>
+<wire x1="58.42" y1="68.58" x2="58.42" y2="33.02" width="0.1524" layer="91"/>
+<pinref part="L_DRIVE" gate="G$1" pin="G/LOW"/>
+<wire x1="58.42" y1="33.02" x2="114.3" y2="33.02" width="0.1524" layer="91"/>
 </segment>
 </net>
 <net name="N$7" class="0">
 <segment>
-<pinref part="ETH1" gate="G$1" pin="7"/>
-<wire x1="53.34" y1="68.58" x2="91.44" y2="68.58" width="0.1524" layer="91"/>
-<wire x1="91.44" y1="68.58" x2="91.44" y2="86.36" width="0.1524" layer="91"/>
-<pinref part="U$1" gate="G$1" pin="P$2"/>
-<wire x1="91.44" y1="86.36" x2="102.87" y2="86.36" width="0.1524" layer="91"/>
-<wire x1="102.87" y1="86.36" x2="102.87" y2="85.09" width="0.1524" layer="91"/>
-</segment>
-</net>
-<net name="N$8" class="0">
-<segment>
-<pinref part="ETH1" gate="G$1" pin="8"/>
-<wire x1="53.34" y1="71.12" x2="86.36" y2="71.12" width="0.1524" layer="91"/>
-<wire x1="86.36" y1="71.12" x2="86.36" y2="91.44" width="0.1524" layer="91"/>
-<pinref part="U$1" gate="G$1" pin="P$1"/>
-<wire x1="86.36" y1="91.44" x2="102.87" y2="91.44" width="0.1524" layer="91"/>
-<wire x1="102.87" y1="91.44" x2="102.87" y2="90.17" width="0.1524" layer="91"/>
+<pinref part="REAR" gate="G$1" pin="3"/>
+<wire x1="53.34" y1="58.42" x2="66.04" y2="58.42" width="0.1524" layer="91"/>
+<wire x1="66.04" y1="58.42" x2="66.04" y2="86.36" width="0.1524" layer="91"/>
+<pinref part="T_DRIVE" gate="G$1" pin="V/SIG"/>
+<wire x1="66.04" y1="86.36" x2="111.76" y2="86.36" width="0.1524" layer="91"/>
 </segment>
 </net>
 </nets>
 </sheet>
-<sheet>
-<plain>
-</plain>
-<instances>
-</instances>
-<busses>
-</busses>
-<nets>
-</nets>
-</sheet>

Commit message: all gerbers generated
Parts:
- added H1, H2, H3, H4: STAND-OFF, SparkFun-Electromechanical:STAND-OFF
Changed lines of the file:
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@@
 <part name="L_SIG" library="TE 2-pin connector" deviceset="2_PIN_TECONNECTOR" device=""/>
 <part name="L_DRIVE" library="TE 2-pin connector" deviceset="2_PIN_TECONNECTOR" device=""/>
+<part name="H1" library="SparkFun-Electromechanical" deviceset="STAND-OFF" device=""/>
+<part name="H2" library="SparkFun-Electromechanical" deviceset="STAND-OFF" device=""/>
+<part name="H3" library="SparkFun-Electromechanical" deviceset="STAND-OFF" device=""/>
+<part name="H4" library="SparkFun-Electromechanical" deviceset="STAND-OFF" device=""/>
 </parts>
 <sheets>
@@
 <instance part="L_SIG" gate="G$1" x="119.38" y="50.8"/>
 <instance part="L_DRIVE" gate="G$1" x="119.38" y="30.48"/>
+<instance part="H1" gate="G$1" x="30.48" y="38.1"/>
+<instance part="H2" gate="G$1" x="38.1" y="38.1"/>
+<instance part="H3" gate="G$1" x="30.48" y="33.02"/>
+<instance part="H4" gate="G$1" x="38.1" y="33.02"/>
 </instances>
 <busses>
