File: rear_light_connect.brd (EAGLE design)
At the start: 48.7 x 79.1 mm, 5 parts

Commit message: all gerbers generated
Parts:
- added H1, H2, H3, H4: STAND-OFF, SparkFun-Electromechanical:STAND-OFF
Changed lines of the file:
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@@
 <element name="R-DRIVE" library="TE 2-pin connector" package="2_PIN_CONNECT" value="2_PIN_TECONNECTOR" x="3.81" y="62.23" rot="R270"/>
 <element name="R_SIG" library="TE 2-pin connector" package="2_PIN_CONNECT" value="2_PIN_TECONNECTOR" x="3.81" y="30.48" rot="R270"/>
+<element name="H1" library="SparkFun-Electromechanical" package="STAND-OFF" value="STAND-OFF" x="4.725" y="1.4"/>
+<element name="H2" library="SparkFun-Electromechanical" package="STAND-OFF" value="STAND-OFF" x="44.275" y="1.575"/>
+<element name="H3" library="SparkFun-Electromechanical" package="STAND-OFF" value="STAND-OFF" x="4.725" y="72.8"/>
+<element name="H4" library="SparkFun-Electromechanical" package="STAND-OFF" value="STAND-OFF" x="44.275" y="72.975"/>
 </elements>
 <signals>
