File: rear_light_connect.sch (EAGLE design)
At the start: 5 parts

Commit message: all gerbers generated
Parts:
- added H1, H2, H3, H4: STAND-OFF, SparkFun-Electromechanical:STAND-OFF
Changed lines of the file:
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@@
 <part name="L_DRIVE" library="TE 2-pin connector" deviceset="2_PIN_TECONNECTOR" device=""/>
 <part name="R-DRIVE" library="TE 2-pin connector" deviceset="2_PIN_TECONNECTOR" device=""/>
+<part name="H1" library="SparkFun-Electromechanical" deviceset="STAND-OFF" device=""/>
+<part name="H2" library="SparkFun-Electromechanical" deviceset="STAND-OFF" device=""/>
+<part name="H3" library="SparkFun-Electromechanical" deviceset="STAND-OFF" device=""/>
+<part name="H4" library="SparkFun-Electromechanical" deviceset="STAND-OFF" device=""/>
 </parts>
 <sheets>
@@
 <instance part="L_DRIVE" gate="G$1" x="119.38" y="50.8"/>
 <instance part="R-DRIVE" gate="G$1" x="119.38" y="30.48"/>
+<instance part="H1" gate="G$1" x="35.56" y="38.1"/>
+<instance part="H2" gate="G$1" x="40.64" y="38.1"/>
+<instance part="H3" gate="G$1" x="48.26" y="38.1"/>
+<instance part="H4" gate="G$1" x="35.56" y="30.48"/>
 </instances>
 <busses>
