File: left board.brd (EAGLE design)
At the start: 100 x 80 mm, 50 parts, among them IC1 LM555D, IC2 LM555D, Q1 10, Q2 10

Commit message: all gerbers generated
Parts:
- added H1, H2, H3, H4: STAND-OFF, SparkFun-Electromechanical:STAND-OFF
- moved L_BLINK 7.00 mm to (101.6, 18.4)
- moved L_DRIVE 4.00 mm to (101.6, 64.6)
Routing:
- net BLINK: track 7.84 -> 10.7 mm
Changed lines of the file:
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@@
 <setting verticaltext="up"/>
 </settings>
-<grid distance="50" unitdist="mil" unit="mil" style="lines" multiple="1" display="no" altdistance="5" altunitdist="mil" altunit="mil"/>
+<grid distance="39.3700787" unitdist="mil" unit="mil" style="lines" multiple="1" display="no" altdistance="5" altunitdist="mil" altunit="mil"/>
 <layers>
 <layer number="1" name="Top" color="4" fill="1" visible="yes" active="yes"/>
@@
 <element name="IC1" library="linear" library_urn="urn:adsk.eagle:library:262" package="SO08" package3d_urn="urn:adsk.eagle:package:16404/2" value="LM555D" x="27.94" y="13.97" rot="MR270"/>
 <element name="IC2" library="linear" library_urn="urn:adsk.eagle:library:262" package="SO08" package3d_urn="urn:adsk.eagle:package:16404/2" value="LM555D" x="66.04" y="13.97" rot="MR270"/>
-<element name="L_BLINK" library="TE 2-pin connector" package="2_PIN_CONNECT" value="2_PIN_TECONNECTOR" x="101.6" y="11.43" rot="R90"/>
-<element name="L_DRIVE" library="TE 2-pin connector" package="2_PIN_CONNECT" value="2_PIN_TECONNECTOR" x="101.6" y="68.58" rot="R90"/>
+<element name="L_BLINK" library="TE 2-pin connector" package="2_PIN_CONNECT" value="2_PIN_TECONNECTOR" x="101.6" y="18.43" rot="R90"/>
+<element name="L_DRIVE" library="TE 2-pin connector" package="2_PIN_CONNECT" value="2_PIN_TECONNECTOR" x="101.6" y="64.58" rot="R90"/>
 <element name="U$1" library="slide switch" package="MYPART3" value="JS_SERIES_SLIDESWITCCH" x="81.28" y="7.62" rot="R90"/>
 <element name="U$2" library="slide switch" package="MYPART3" value="JS_SERIES_SLIDESWITCCH" x="81.28" y="63.5" rot="MR90"/>
@@
 <element name="Q2" library="transistor-power" library_urn="urn:adsk.eagle:library:400" package="TO220BV" package3d_urn="urn:adsk.eagle:package:29484/1" value="10" x="27.94" y="26.67" rot="R270"/>
 <element name="Q1" library="transistor-power" library_urn="urn:adsk.eagle:library:400" package="TO220BV" package3d_urn="urn:adsk.eagle:package:29484/1" value="10" x="60.96" y="21.59" rot="R270"/>
+<element name="H1" library="SparkFun-Electromechanical" package="STAND-OFF" value="STAND-OFF" x="5" y="5"/>
+<element name="H2" library="SparkFun-Electromechanical" package="STAND-OFF" value="STAND-OFF" x="95" y="5"/>
+<element name="H3" library="SparkFun-Electromechanical" package="STAND-OFF" value="STAND-OFF" x="4" y="76"/>
+<element name="H4" library="SparkFun-Electromechanical" package="STAND-OFF" value="STAND-OFF" x="96" y="76"/>
 </elements>
 <signals>
@@
 <contactref element="L_BLINK" pad="V/SIG"/>
 <contactref element="U$1" pad="IN"/>
-<wire x1="81.28" y1="7.62" x2="88.46" y2="7.62" width="0.4064" layer="1"/>
-<wire x1="88.46" y1="7.62" x2="88.93" y2="8.09" width="0.4064" layer="1"/>
+<wire x1="81.28" y1="7.62" x2="81.46" y2="7.62" width="0.6096" layer="16"/>
+<wire x1="81.46" y1="7.62" x2="88.93" y2="15.09" width="0.6096" layer="16"/>
 </signal>
 <signal name="DRIVE">
@@
 <contactref element="U$2" pad="IN"/>
 <wire x1="81.28" y1="63.5" x2="87.19" y2="63.5" width="0.4064" layer="1"/>
-<wire x1="87.19" y1="63.5" x2="88.93" y2="65.24" width="0.4064" layer="1"/>
+<wire x1="87.19" y1="63.5" x2="88.93" y2="61.24" width="0.4064" layer="1"/>
 </signal>
 <signal name="B_OUT">

Commit message: via gerbers generated
via boards completed and gerbers generated
Parts:
- removed Q1, Q2: 10, transistor-power:TO220BV
- added Q3, Q4: BSS101, transistor-fet:TO92
Connections:
- net B_BLINK: now also Q3.1; no longer Q2.S
- net B_OUT: now also Q3.2; no longer Q2.G
- net D_BLINK: now also Q4.1; no longer Q1.S
- net D_OUT: now also Q4.2; no longer Q1.G
- net N$1: now also Q3.3; no longer Q2.D
- net N$11: now also Q4.3; no longer Q1.D
Routing:
- net B_BLINK: track 76.8 -> 91.5 mm, vias 2 -> 3
- net D_OUT: track 59.5 -> 65.1 mm
- net B_OUT: track 71.4 -> 76.5 mm
- net D_BLINK: track 67.1 -> 65.6 mm
- net N$1: track 5.45 -> 4.47 mm
Changed lines of the file:
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@@
 <layers>
 <layer number="1" name="Top" color="4" fill="1" visible="yes" active="yes"/>
+<layer number="2" name="Route2" color="1" fill="3" visible="yes" active="yes"/>
+<layer number="3" name="Route3" color="4" fill="3" visible="yes" active="yes"/>
+<layer number="4" name="Route4" color="1" fill="4" visible="yes" active="yes"/>
+<layer number="5" name="Route5" color="4" fill="4" visible="yes" active="yes"/>
+<layer number="6" name="Route6" color="1" fill="8" visible="yes" active="yes"/>
+<layer number="7" name="Route7" color="4" fill="8" visible="yes" active="yes"/>
+<layer number="8" name="Route8" color="1" fill="2" visible="yes" active="yes"/>
+<layer number="9" name="Route9" color="4" fill="2" visible="yes" active="yes"/>
+<layer number="10" name="Route10" color="1" fill="7" visible="yes" active="yes"/>
+<layer number="11" name="Route11" color="4" fill="7" visible="yes" active="yes"/>
+<layer number="12" name="Route12" color="1" fill="5" visible="yes" active="yes"/>
+<layer number="13" name="Route13" color="4" fill="5" visible="yes" active="yes"/>
+<layer number="14" name="Route14" color="1" fill="6" visible="yes" active="yes"/>
+<layer number="15" name="Route15" color="4" fill="6" visible="yes" active="yes"/>
 <layer number="16" name="Bottom" color="1" fill="1" visible="yes" active="yes"/>
 <layer number="17" name="Pads" color="2" fill="1" visible="yes" active="yes"/>
@@
 <attribute name="PROD_ID" value="RES-12428" x="66.04" y="5.08" size="1.778" layer="28" rot="MR180" display="off"/>
 </element>
-<element name="Q2" library="transistor-power" library_urn="urn:adsk.eagle:library:400" package="TO220BV" package3d_urn="urn:adsk.eagle:package:29484/1" value="10" x="27.94" y="26.67" rot="R270"/>
-<element name="Q1" library="transistor-power" library_urn="urn:adsk.eagle:library:400" package="TO220BV" package3d_urn="urn:adsk.eagle:package:29484/1" value="10" x="60.96" y="21.59" rot="R270"/>
 <element name="H1" library="SparkFun-Electromechanical" package="STAND-OFF" value="STAND-OFF" x="5" y="5"/>
 <element name="H2" library="SparkFun-Electromechanical" package="STAND-OFF" value="STAND-OFF" x="95" y="5"/>
 <element name="H3" library="SparkFun-Electromechanical" package="STAND-OFF" value="STAND-OFF" x="4" y="76"/>
 <element name="H4" library="SparkFun-Electromechanical" package="STAND-OFF" value="STAND-OFF" x="96" y="76"/>
+<element name="Q3" library="transistor-fet" library_urn="urn:adsk.eagle:library:396" package="TO92" package3d_urn="urn:adsk.eagle:package:28523/1" value="BSS101" x="25" y="25" rot="MR180"/>
+<element name="Q4" library="transistor-fet" library_urn="urn:adsk.eagle:library:396" package="TO92" package3d_urn="urn:adsk.eagle:package:28523/1" value="BSS101" x="59" y="20" rot="MR180"/>
 </elements>
 <signals>
@@
 <contactref element="U$1" pad="OUT2"/>
 <contactref element="R12" pad="1"/>
-<contactref element="Q2" pad="G"/>
 <wire x1="81.28" y1="10.8204" x2="56.30815" y2="10.8204" width="0.4064" layer="1"/>
 <wire x1="56.30815" y1="10.8204" x2="56.18395" y2="10.6962" width="0.4064" layer="1"/>
 <wire x1="56.18395" y1="10.6962" x2="46.22155" y2="10.6962" width="0.4064" layer="1"/>
 <wire x1="46.22155" y1="10.6962" x2="33.32395" y2="23.5938" width="0.4064" layer="1"/>
-<wire x1="31.0162" y1="23.5938" x2="25.4" y2="29.21" width="0.4064" layer="1"/>
-<wire x1="33.32395" y1="23.5938" x2="31.0162" y2="23.5938" width="0.4064" layer="1"/>
-<wire x1="25.4" y1="29.21" x2="21.22" y2="29.21" width="0.4064" layer="1"/>
-<wire x1="21.22" y1="29.21" x2="18.68" y2="31.75" width="0.4064" layer="1"/>
+<wire x1="21.22" y1="29.21" x2="21.215" y2="29.215" width="0.4064" layer="1"/>
+<contactref element="Q3" pad="2"/>
+<wire x1="21.215" y1="29.215" x2="18.68" y2="31.75" width="0.4064" layer="1"/>
+<wire x1="25.4988" y1="23.5938" x2="25" y2="23.095" width="0.4064" layer="1"/>
+<wire x1="29.892503125" y1="23.5938" x2="33.32395" y2="23.5938" width="0.4064" layer="1"/>
+<wire x1="29.892503125" y1="23.5938" x2="25.4988" y2="23.5938" width="0.4064" layer="1"/>
+<wire x1="21.215" y1="29.215" x2="24.271303125" y2="29.215" width="0.4064" layer="1"/>
+<wire x1="24.271303125" y1="29.215" x2="29.892503125" y2="23.5938" width="0.4064" layer="1"/>
 </signal>
 <signal name="D_OUT">
@@
 <wire x1="78.74" y1="64.1604" x2="81.28" y2="66.7004" width="0.4064" layer="16"/>
 <wire x1="78.74" y1="43.18" x2="78.74" y2="64.1604" width="0.4064" layer="16"/>
-<contactref element="Q1" pad="G"/>
-<wire x1="58.42" y1="24.13" x2="58.76" y2="24.13" width="0.4064" layer="16"/>
-<wire x1="58.76" y1="24.13" x2="62.4" y2="20.49" width="0.4064" layer="16"/>
+<wire x1="58.76" y1="24.13" x2="58.945" y2="23.945" width="0.4064" layer="16"/>
+<contactref element="Q4" pad="2"/>
+<wire x1="58.945" y1="23.945" x2="62.4" y2="20.49" width="0.4064" layer="16"/>
+<wire x1="58.945" y1="23.945" x2="58.945" y2="18.15" width="0.508" layer="16"/>
+<wire x1="58.945" y1="18.15" x2="59" y2="18.095" width="0.508" layer="16"/>
 </signal>
 <signal name="D_BLINK">
@@
 <wire x1="68.58" y1="30.48" x2="81.28" y2="43.18" width="0.4064" layer="1"/>
 <wire x1="81.28" y1="43.18" x2="81.28" y2="60.2996" width="0.4064" layer="1"/>
-<contactref element="Q1" pad="S"/>
 <wire x1="64.2338" y1="21.28605" x2="64.2338" y2="21.9538" width="0.4064" layer="16"/>
-<wire x1="58.42" y1="19.05" x2="61.99775" y2="19.05" width="0.4064" layer="16"/>
 <wire x1="61.99775" y1="19.05" x2="64.2338" y2="21.28605" width="0.4064" layer="16"/>
 <wire x1="64.2338" y1="21.9538" x2="66.04" y2="23.76" width="0.4064" layer="16"/>
+<contactref element="Q4" pad="1"/>
+<wire x1="60.27" y1="20" x2="61.04775" y2="20" width="0.508" layer="16"/>
+<wire x1="61.04775" y1="20" x2="61.99775" y2="19.05" width="0.508" layer="16"/>
 </signal>
 <signal name="B_BLINK">
@@
 <wire x1="45.455" y1="13.335" x2="45.72" y2="13.07" width="0.4064" layer="16"/>
 <wire x1="31.78729375" y1="13.9494" x2="31.9956" y2="14.15770625" width="0.4064" layer="16"/>
-<wire x1="31.9956" y1="14.15770625" x2="31.9956" y2="15.05229375" width="0.4064" layer="16"/>
+<wire x1="31.9956" y1="15.05229375" x2="31.9956" y2="14.15770625" width="0.4064" layer="16"/>
 <wire x1="31.9956" y1="15.05229375" x2="31.78729375" y2="15.2606" width="0.4064" layer="16"/>
 <wire x1="30.54" y1="13.335" x2="31.1544" y2="13.9494" width="0.4064" layer="16"/>
@@
 <wire x1="33.02" y1="19.05" x2="33.02" y2="18.28704375" width="0.4064" layer="16"/>
 <wire x1="33.02" y1="18.28704375" x2="30.573978125" y2="15.841021875" width="0.4064" layer="16"/>
-<contactref element="Q2" pad="S"/>
-<wire x1="25.4" y1="24.13" x2="31.75" y2="24.13" width="0.4064" layer="16"/>
 <wire x1="31.75" y1="24.13" x2="33.02" y2="22.86" width="0.4064" layer="16"/>
+<contactref element="Q3" pad="1"/>
+<wire x1="30.54" y1="13.335" x2="32.335" y2="13.335" width="0.4064" layer="16"/>
+<wire x1="32.335" y1="13.335" x2="34" y2="15" width="0.4064" layer="16"/>
+<via x="34" y="15" extent="1-16" drill="0.35"/>
+<wire x1="24.57915625" y1="22.079" x2="23.984" y2="22.67415625" width="0.4064" layer="1"/>
+<wire x1="23.984" y1="22.67415625" x2="23.984" y2="23.51584375" width="0.4064" layer="1"/>
+<wire x1="25.4226" y1="24.1526" x2="26.27" y2="25" width="0.4064" layer="1"/>
+<wire x1="34" y1="15" x2="26.921" y2="22.079" width="0.4064" layer="1"/>
+<wire x1="26.921" y1="22.079" x2="24.57915625" y2="22.079" width="0.4064" layer="1"/>
+<wire x1="23.984" y1="23.51584375" x2="24.62075625" y2="24.1526" width="0.4064" layer="1"/>
+<wire x1="24.62075625" y1="24.1526" x2="25.4226" y2="24.1526" width="0.4064" layer="1"/>
 </signal>
 <signal name="N$9">
@@
 <contactref element="R14" pad="1"/>
 <wire x1="54.81" y1="22.69" x2="54.61" y2="22.49" width="0.4064" layer="16"/>
-<contactref element="Q1" pad="D"/>
-<wire x1="54.61" y1="22.49" x2="57.52" y2="22.49" width="0.4064" layer="16"/>
-<wire x1="57.52" y1="22.49" x2="58.42" y2="21.59" width="0.4064" layer="16"/>
+<contactref element="Q4" pad="3"/>
+<wire x1="54.61" y1="22.49" x2="55.24" y2="22.49" width="0.508" layer="16"/>
+<wire x1="55.24" y1="22.49" x2="57.73" y2="20" width="0.508" layer="16"/>
 </signal>
 <signal name="N$1">
 <contactref element="R11" pad="2"/>
-<contactref element="Q2" pad="D"/>
-<wire x1="19.95" y1="26.67" x2="25.4" y2="26.67" width="0.4064" layer="16"/>
+<contactref element="Q3" pad="3"/>
+<wire x1="19.95" y1="26.67" x2="22.06" y2="26.67" width="0.508" layer="16"/>
+<wire x1="22.06" y1="26.67" x2="23.73" y2="25" width="0.508" layer="16"/>
 </signal>
 <signal name="N$12">
