File: front_light_via.brd (EAGLE design)
At the start: 48.7 x 79.1 mm, 9 parts

Commit message: via gerbers generated
via boards completed and gerbers generated
Parts:
- removed ETH1: ETHERNET, ETHERNET:A122645-ND
- removed L_DRIVE, L_SIG, R-DRIVE, R_SIG: 2_PIN_TECONNECTOR, TE 2-pin connector:2_PIN_CONNECT
- added BLINK_L, BLINK_R, DRIVING_L, DRIVING_R: 2_PIN_TECONNECTOR, TE 2-pin connector:2_PIN_CONNECT
- added FRONT: ETHERNET, ETHERNET:A122645-ND
- moved H2 12.2 mm to (56.4, 3.50)
- moved H4 12.1 mm to (55.8, 69.3)
- moved H3 3.10 mm to (3.85, 69.8)
- moved H1 2.67 mm to (3.33, 3.67)
Connections:
- removed net N$2: ETH1.P$2, R-DRIVE.G/LOW
- removed net N$4: ETH1.P$4, L_DRIVE.G/LOW
- removed net N$6: ETH1.P$6, R_SIG.G/LOW
- removed net N$8: ETH1.P$8, L_SIG.G/LOW
- new net BLIINK_R: BLINK_R.G/LOW, FRONT.P$4
- new net BLINK_L: BLINK_L.G/LOW, FRONT.P$2
- new net DRIVING_L: DRIVING_L.G/LOW, FRONT.P$8
- new net DRIVING_R: DRIVING_R.G/LOW, FRONT.P$6
- net N$1: now also BLINK_L.V/SIG, FRONT.P$1; no longer ETH1.P$1, R-DRIVE.V/SIG
- net N$3: now also BLINK_R.V/SIG, FRONT.P$3; no longer ETH1.P$3, L_DRIVE.V/SIG
- net N$5: now also DRIVING_R.V/SIG, FRONT.P$5; no longer ETH1.P$5, R_SIG.V/SIG
- net N$7: now also DRIVING_L.V/SIG, FRONT.P$7; no longer ETH1.P$7, L_SIG.V/SIG
Routing:
- net N$6: track 73.5 -> 0.00 mm
- net DRIVING_L: track 0.00 -> 48.2 mm, vias 0 -> 1
- net BLINK_L: track 0.00 -> 44.7 mm
- net BLIINK_R: track 0.00 -> 43.5 mm
- net DRIVING_R: track 0.00 -> 39.5 mm
- net N$8: track 36.7 -> 0.00 mm
- net N$2: track 27.0 -> 0.00 mm
- net N$5: track 33.4 -> 56.7 mm, vias 0 -> 1
- net N$4: track 21.5 -> 0.00 mm
- net N$1: track 30.7 -> 48.2 mm
- net N$3: track 36.9 -> 49.0 mm
- net N$7: track 47.0 -> 48.0 mm
Other:
- board size 48.7 x 79.1 mm -> 60 x 73 mm
- board text added: "DRIVE_L"
- board text added: "DRIVE_R"
- board text added: "L_sig"
- board text added: "R_sig"

Commit message: added reverse polairity protection
Parts:
- removed BLINK_L, BLINK_R, DRIVING_L, DRIVING_R: 2_PIN_TECONNECTOR, TE 2-pin connector:2_PIN_CONNECT
- added U$1, U$2, U$3, U$4: 2_PIN_TECONNECTOR, TE 2-pin connector:2_PIN_CONNECT
Connections:
- net BLIINK_R: now also U$3.G/LOW; no longer BLINK_R.G/LOW
- net BLINK_L: now also U$4.G/LOW; no longer BLINK_L.G/LOW
- net DRIVING_L: now also U$1.G/LOW; no longer DRIVING_L.G/LOW
- net DRIVING_R: now also U$2.G/LOW; no longer DRIVING_R.G/LOW
- net N$1: now also U$4.V/SIG; no longer BLINK_L.V/SIG
- net N$3: now also U$3.V/SIG; no longer BLINK_R.V/SIG
- net N$5: now also U$2.V/SIG; no longer DRIVING_R.V/SIG
- net N$7: now also U$1.V/SIG; no longer DRIVING_L.V/SIG
Routing:
- net DRIVING_R: track 39.5 -> 40.5 mm
- net BLINK_L: track 44.7 -> 45.6 mm
- net N$7: track 48.0 -> 48.8 mm
- net N$3: track 49.0 -> 49.7 mm
Changed lines of the file:
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@@
 <?xml version="1.0" encoding="utf-8"?>
 <!DOCTYPE eagle SYSTEM "eagle.dtd">
-<eagle version="8.6.0">
+<eagle version="8.6.1">
 <drawing>
 <settings>
@@
 <attribute name="VALUE" x="43.56" y="41.255" size="1.27" layer="21" rot="R90"/>
 </element>
-<element name="BLINK_R" library="TE 2-pin connector" package="2_PIN_CONNECT" value="2_PIN_TECONNECTOR" x="-0.04" y="29.315" rot="R270"/>
-<element name="DRIVING_L" library="TE 2-pin connector" package="2_PIN_CONNECT" value="2_PIN_TECONNECTOR" x="0.135" y="13.795" rot="R270"/>
-<element name="BLINK_L" library="TE 2-pin connector" package="2_PIN_CONNECT" value="2_PIN_TECONNECTOR" x="-0.04" y="59.08" smashed="yes" rot="R270"/>
-<element name="DRIVING_R" library="TE 2-pin connector" package="2_PIN_CONNECT" value="2_PIN_TECONNECTOR" x="0.135" y="44.48" smashed="yes" rot="R270"/>
 <element name="H1" library="SparkFun-Electromechanical" package="STAND-OFF" value="STAND-OFF" x="3.325" y="3.675"/>
 <element name="H2" library="SparkFun-Electromechanical" package="STAND-OFF" value="STAND-OFF" x="56.35" y="3.5"/>
 <element name="H3" library="SparkFun-Electromechanical" package="STAND-OFF" value="STAND-OFF" x="3.85" y="69.825"/>
 <element name="H4" library="SparkFun-Electromechanical" package="STAND-OFF" value="STAND-OFF" x="55.825" y="69.3"/>
+<element name="U$1" library="TE 2-pin connector" package="2_PIN_CONNECT" value="2_PIN_TECONNECTOR" x="0" y="13.475" rot="R270"/>
+<element name="U$2" library="TE 2-pin connector" package="2_PIN_CONNECT" value="2_PIN_TECONNECTOR" x="0.175" y="45.675" rot="R270"/>
+<element name="U$3" library="TE 2-pin connector" package="2_PIN_CONNECT" value="2_PIN_TECONNECTOR" x="0" y="28.875" rot="R270"/>
+<element name="U$4" library="TE 2-pin connector" package="2_PIN_CONNECT" value="2_PIN_TECONNECTOR" x="0" y="60.2" rot="R270"/>
 </elements>
 <signals>
 <signal name="N$1">
 <contactref element="FRONT" pad="P$1"/>
-<contactref element="BLINK_L" pad="V/SIG"/>
 <wire x1="52.45" y1="42.295" x2="32.325" y2="62.42" width="0.508" layer="1"/>
-<wire x1="32.325" y1="62.42" x2="12.63" y2="62.42" width="0.508" layer="1"/>
+<contactref element="U$4" pad="V/SIG"/>
+<wire x1="32.325" y1="62.42" x2="12.82" y2="62.42" width="0.508" layer="1"/>
+<wire x1="12.82" y1="62.42" x2="12.67" y2="62.27" width="0.508" layer="1"/>
 </signal>
 <signal name="BLINK_L">
 <contactref element="FRONT" pad="P$2"/>
-<contactref element="BLINK_L" pad="G/LOW"/>
 <wire x1="50.67" y1="41.275" x2="47.0104" y2="44.9346" width="0.508" layer="1"/>
 <wire x1="47.0104" y1="44.9346" x2="47.0104" y2="46.05565625" width="0.508" layer="1"/>
-<wire x1="47.0104" y1="46.05565625" x2="37.32605625" y2="55.74" width="0.508" layer="1"/>
-<wire x1="37.32605625" y1="55.74" x2="12.63" y2="55.74" width="0.508" layer="1"/>
+<contactref element="U$4" pad="G/LOW"/>
+<wire x1="34.93605625" y1="58.13" x2="12.67" y2="58.13" width="0.508" layer="1"/>
+<wire x1="47.0104" y1="46.05565625" x2="34.93605625" y2="58.13" width="0.508" layer="1"/>
 </signal>
 <signal name="N$3">
 <contactref element="FRONT" pad="P$3"/>
-<contactref element="BLINK_R" pad="V/SIG"/>
 <wire x1="53.6104" y1="38.69565625" x2="53.6104" y2="35.69434375" width="0.508" layer="16"/>
 <wire x1="52.45" y1="40.255" x2="52.45" y2="39.85605625" width="0.508" layer="16"/>
@@
 <wire x1="53.6104" y1="35.69434375" x2="51.91065625" y2="33.9946" width="0.508" layer="16"/>
 <wire x1="51.91065625" y1="33.9946" x2="50.18934375" y2="33.9946" width="0.508" layer="16"/>
-<wire x1="28.875" y1="36.05" x2="25.48" y2="32.655" width="0.508" layer="16"/>
-<wire x1="25.48" y1="32.655" x2="12.63" y2="32.655" width="0.508" layer="16"/>
+<contactref element="U$3" pad="V/SIG"/>
+<wire x1="23.77" y1="30.945" x2="12.67" y2="30.945" width="0.508" layer="16"/>
+<wire x1="28.875" y1="36.05" x2="23.77" y2="30.945" width="0.508" layer="16"/>
 </signal>
 <signal name="BLIINK_R">
 <contactref element="FRONT" pad="P$4"/>
-<contactref element="BLINK_R" pad="G/LOW"/>
 <wire x1="50.67" y1="39.235" x2="46.7404" y2="35.3054" width="0.508" layer="1"/>
 <wire x1="46.7404" y1="35.3054" x2="45.36934375" y2="35.3054" width="0.508" layer="1"/>
-<wire x1="36.03894375" y1="25.975" x2="12.63" y2="25.975" width="0.508" layer="1"/>
 <wire x1="45.36934375" y1="35.3054" x2="36.03894375" y2="25.975" width="0.508" layer="1"/>
+<contactref element="U$3" pad="G/LOW"/>
+<wire x1="36.03894375" y1="25.975" x2="13.5" y2="25.975" width="0.508" layer="1"/>
+<wire x1="13.5" y1="25.975" x2="12.67" y2="26.805" width="0.508" layer="1"/>
 </signal>
 <signal name="N$5">
 <contactref element="FRONT" pad="P$5"/>
-<contactref element="DRIVING_R" pad="V/SIG"/>
 <via x="49.35" y="47.775" extent="1-16" drill="0.35"/>
 <wire x1="57.885" y1="43.86585" x2="57.885" y2="46.26415" width="0.508" layer="1"/>
@@
 <wire x1="50.006075" y1="47.775" x2="49.35" y2="47.775" width="0.508" layer="1"/>
 <wire x1="49.35" y1="47.775" x2="12.85" y2="47.775" width="0.508" layer="16"/>
-<wire x1="12.85" y1="47.775" x2="12.805" y2="47.82" width="0.508" layer="16"/>
+<contactref element="U$2" pad="V/SIG"/>
+<wire x1="12.845" y1="47.745" x2="12.85" y2="47.775" width="0" layer="19" extent="16-16"/>
 </signal>
 <signal name="DRIVING_R">
 <contactref element="FRONT" pad="P$6"/>
-<contactref element="DRIVING_R" pad="G/LOW"/>
-<wire x1="50.67" y1="37.195" x2="46.725" y2="41.14" width="0.508" layer="16"/>
-<wire x1="46.725" y1="41.14" x2="12.805" y2="41.14" width="0.508" layer="16"/>
+<contactref element="U$2" pad="G/LOW"/>
+<wire x1="45.7404" y1="42.1246" x2="45.36934375" y2="42.1246" width="0.508" layer="16"/>
+<wire x1="43.88894375" y1="43.605" x2="12.845" y2="43.605" width="0.508" layer="16"/>
+<wire x1="45.36934375" y1="42.1246" x2="43.88894375" y2="43.605" width="0.508" layer="16"/>
+<wire x1="50.67" y1="37.195" x2="45.7404" y2="42.1246" width="0.508" layer="16"/>
 </signal>
 <signal name="N$7">
 <contactref element="FRONT" pad="P$7"/>
-<contactref element="DRIVING_L" pad="V/SIG"/>
 <wire x1="52.45" y1="36.175" x2="51.8304" y2="35.5554" width="0.508" layer="1"/>
 <wire x1="51.8304" y1="35.5554" x2="51.8304" y2="34.67434375" width="0.508" layer="1"/>
 <wire x1="51.8304" y1="34.67434375" x2="34.29105625" y2="17.135" width="0.508" layer="1"/>
-<wire x1="34.29105625" y1="17.135" x2="12.805" y2="17.135" width="0.508" layer="1"/>
+<contactref element="U$1" pad="V/SIG"/>
+<wire x1="34.29105625" y1="17.135" x2="14.26" y2="17.135" width="0.508" layer="1"/>
+<wire x1="14.26" y1="17.135" x2="12.67" y2="15.545" width="0.508" layer="1"/>
 </signal>
 <signal name="DRIVING_L">
 <contactref element="FRONT" pad="P$8"/>
-<contactref element="DRIVING_L" pad="G/LOW"/>
 <via x="28.175" y="18.55" extent="1-16" drill="0.35"/>
 <wire x1="50.67" y1="35.155" x2="47.0104" y2="31.4954" width="0.508" layer="1"/>
@@
 <wire x1="34.18605625" y1="18.55" x2="28.175" y2="18.55" width="0.508" layer="1"/>
 <wire x1="28.175" y1="18.55" x2="20.9" y2="18.55" width="0.508" layer="16"/>
-<wire x1="20.9" y1="18.55" x2="12.805" y2="10.455" width="0.508" layer="16"/>
+<contactref element="U$1" pad="G/LOW"/>
+<wire x1="20.9" y1="18.55" x2="13.755" y2="11.405" width="0.508" layer="16"/>
+<wire x1="13.755" y1="11.405" x2="12.67" y2="11.405" width="0.508" layer="16"/>
 </signal>
 </signals>
